Commit message: Update fixed-wing URDF and add main flight launch file

File: ros_ws/src/uav_description/urdf/fixed_wing/airplane.xacro (robot description, xacro)
@@ -2,7 +2,7 @@
 <robot name="airplane" xmlns:xacro="http://ros.org/wiki/xacro">
     <!-- Add the Gazebo xacro file-->
-    <xacro:include filename="$(find plane_description)/urdf/fixed_wing/airplane_gazebo.xacro"/>
+    <xacro:include filename="$(find uav_description)/urdf/fixed_wing/airplane_gazebo.xacro"/>
     <!-- Add the for spawner file-->
-    <xacro:include filename="$(find plane_description)/urdf/fixed_wing/add_fog.xacro"/>
+    <xacro:include filename="$(find uav_description)/urdf/fixed_wing/add_fog.xacro"/>
     <xacro:macro name="airplane" params="robot_scale robot_name camera_num world_name initial_alt fog_lifetime fog_rate enable_fog">
         <!-- LINK SECTIONS OF THE AIRPLANE-->
@@ -20,11 +20,11 @@
             <collision name="collision">
                 <geometry>
-                <mesh filename="file://$(find plane_description)/meshes/Cessna/body.dae"
-                        scale="${robot_scale} ${robot_scale} ${robot_scale}"/>
-                </geometry>
-            </collision>
-            <visual name="visual">
-                <geometry>
-                <mesh filename="file://$(find plane_description)/meshes/Cessna/body.dae"
+                <mesh filename="file://$(find uav_description)/meshes/Cessna/body.dae"
+                        scale="${robot_scale} ${robot_scale} ${robot_scale}"/>
+                </geometry>
+            </collision>
+            <visual name="visual">
+                <geometry>
+                <mesh filename="file://$(find uav_description)/meshes/Cessna/body.dae"
                         scale="${robot_scale} ${robot_scale} ${robot_scale}"/>
                 </geometry>
@@ -41,11 +41,11 @@
             <collision name="collision">
                 <geometry>
-                <mesh filename="file://$(find plane_description)/meshes/Cessna/left_aileron.dae"
-                        scale="${robot_scale} ${robot_scale} ${robot_scale}"/>
-                </geometry>
-            </collision>
-            <visual name="visual">
-                <geometry>
-                <mesh filename="file://$(find plane_description)/meshes/Cessna/left_aileron.dae"
+                <mesh filename="file://$(find uav_description)/meshes/Cessna/left_aileron.dae"
+                        scale="${robot_scale} ${robot_scale} ${robot_scale}"/>
+                </geometry>
+            </collision>
+            <visual name="visual">
+                <geometry>
+                <mesh filename="file://$(find uav_description)/meshes/Cessna/left_aileron.dae"
                         scale="${robot_scale} ${robot_scale} ${robot_scale}"/>
                 </geometry>
@@ -62,11 +62,11 @@
             <collision name="collision">
                 <geometry>
-                <mesh filename="file://$(find plane_description)/meshes/Cessna/left_flap.dae"
-                        scale="${robot_scale} ${robot_scale} ${robot_scale}"/>
-                </geometry>
-            </collision>
-            <visual name="visual">
-                <geometry>
-                <mesh filename="file://$(find plane_description)/meshes/Cessna/left_flap.dae"
+                <mesh filename="file://$(find uav_description)/meshes/Cessna/left_flap.dae"
+                        scale="${robot_scale} ${robot_scale} ${robot_scale}"/>
+                </geometry>
+            </collision>
+            <visual name="visual">
+                <geometry>
+                <mesh filename="file://$(find uav_description)/meshes/Cessna/left_flap.dae"
                         scale="${robot_scale} ${robot_scale} ${robot_scale}"/>
                 </geometry>
@@ -83,11 +83,11 @@
             <collision name="collision">
                 <geometry>
-                <mesh filename="file://$(find plane_description)/meshes/Cessna/right_aileron.dae"
-                        scale="${robot_scale} ${robot_scale} ${robot_scale}"/>
-                </geometry>
-            </collision>
-            <visual name="visual">
-                <geometry>
-                <mesh filename="file://$(find plane_description)/meshes/Cessna/right_aileron.dae"
+                <mesh filename="file://$(find uav_description)/meshes/Cessna/right_aileron.dae"
+                        scale="${robot_scale} ${robot_scale} ${robot_scale}"/>
+                </geometry>
+            </collision>
+            <visual name="visual">
+                <geometry>
+                <mesh filename="file://$(find uav_description)/meshes/Cessna/right_aileron.dae"
                         scale="${robot_scale} ${robot_scale} ${robot_scale}"/>
                 </geometry>
@@ -104,11 +104,11 @@
             <collision name="collision">
                 <geometry>
-                <mesh filename="file://$(find plane_description)/meshes/Cessna/right_flap.dae"
-                        scale="${robot_scale} ${robot_scale} ${robot_scale}"/>
-                </geometry>
-            </collision>
-            <visual name="visual">
-                <geometry>
-                <mesh filename="file://$(find plane_description)/meshes/Cessna/right_flap.dae"
+                <mesh filename="file://$(find uav_description)/meshes/Cessna/right_flap.dae"
+                        scale="${robot_scale} ${robot_scale} ${robot_scale}"/>
+                </geometry>
+            </collision>
+            <visual name="visual">
+                <geometry>
+                <mesh filename="file://$(find uav_description)/meshes/Cessna/right_flap.dae"
                         scale="${robot_scale} ${robot_scale} ${robot_scale}"/>
                 </geometry>
@@ -125,11 +125,11 @@
             <collision name="collision">
                 <geometry>
-                <mesh filename="file://$(find plane_description)/meshes/Cessna/elevators.dae"
-                        scale="${robot_scale} ${robot_scale} ${robot_scale}"/>
-                </geometry>
-            </collision>
-            <visual name="visual">
-                <geometry>
-                <mesh filename="file://$(find plane_description)/meshes/Cessna/elevators.dae"
+                <mesh filename="file://$(find uav_description)/meshes/Cessna/elevators.dae"
+                        scale="${robot_scale} ${robot_scale} ${robot_scale}"/>
+                </geometry>
+            </collision>
+            <visual name="visual">
+                <geometry>
+                <mesh filename="file://$(find uav_description)/meshes/Cessna/elevators.dae"
                         scale="${robot_scale} ${robot_scale} ${robot_scale}"/>
                 </geometry>
@@ -146,11 +146,11 @@
             <collision name="collision">
                 <geometry>
-                <mesh filename="file://$(find plane_description)/meshes/Cessna/rudder.dae"
-                        scale="${robot_scale} ${robot_scale} ${robot_scale}"/>
-                </geometry>
-            </collision>
-            <visual name="visual">
-                <geometry>
-                <mesh filename="file://$(find plane_description)/meshes/Cessna/rudder.dae"
+                <mesh filename="file://$(find uav_description)/meshes/Cessna/rudder.dae"
+                        scale="${robot_scale} ${robot_scale} ${robot_scale}"/>
+                </geometry>
+            </collision>
+            <visual name="visual">
+                <geometry>
+                <mesh filename="file://$(find uav_description)/meshes/Cessna/rudder.dae"
                         scale="${robot_scale} ${robot_scale} ${robot_scale}"/>
                 </geometry>
@@ -167,11 +167,11 @@
             <collision name="collision">
                 <geometry>
-                <mesh filename="file://$(find plane_description)/meshes/Cessna/cessna_prop.dae"
-                        scale="${robot_scale} ${robot_scale} ${robot_scale}"/>
-                </geometry>
-            </collision>
-            <visual name="visual">
-                <geometry>
-                <mesh filename="file://$(find plane_description)/meshes/Cessna/cessna_prop.dae"
+                <mesh filename="file://$(find uav_description)/meshes/Cessna/cessna_prop.dae"
+                        scale="${robot_scale} ${robot_scale} ${robot_scale}"/>
+                </geometry>
+            </collision>
+            <visual name="visual">
+                <geometry>
+                <mesh filename="file://$(find uav_description)/meshes/Cessna/cessna_prop.dae"
                         scale="${robot_scale} ${robot_scale} ${robot_scale}"/>
                 </geometry>

File: ros_ws/src/uav_description/urdf/fixed_wing/main_fixed_wing.xacro (robot description, xacro)
@@ -1,5 +1,5 @@
 <?xml version="1.0"?>
 <robot xmlns:xacro="http://www.ros.org/wiki/xacro" name="main_airplane">
-    <xacro:include filename="$(find plane_description)/urdf/fixed_wing/airplane.xacro"/>
+    <xacro:include filename="$(find uav_description)/urdf/fixed_wing/airplane.xacro"/>
     <xacro:arg name="robot_name" default="airplane_1"/>
     <xacro:arg name="robot_scale" default="1.0"/>

Commit message: Integrate ADS-B EKF plugin into airplane URDF and update GNSS submodule

File: ros_ws/src/uav_description/urdf/fixed_wing/airplane.xacro (robot description, xacro)
@@ -248,4 +248,18 @@
             </inertial>
         </link>
+        <!--IMU Link for teh ADS-B Reciever-->
+        <link name="imu_link">
+            <visual>
+                <origin xyz="0 0 0" rpy="0 0 0"/>
+                <geometry>
+                    <box size="${0.02 * robot_scale} ${0.02 * robot_scale} ${0.02 * robot_scale}"/>
+                </geometry>
+            </visual>
+            <inertial>
+                <mass value="${0.001 * robot_scale}" />
+                <origin xyz="0 0 0" rpy="0 0 0"/>
+                <inertia ixx="0.00000015" ixy="0" ixz="0" iyy="0.00000015" iyz="0" izz="0.00000015" />
+            </inertial>
+        </link>
         <!-- Joint of the sensors or plugin requirements -->
         <!-- Frontal camera fized joint-->
@@ -255,9 +269,15 @@
             <child link="frontal_camera_link"/>
         </joint>
-        <!-- GNSS Lidar link-->
+        <!-- GNSS Lidar joint-->
         <joint name="lidar_link_joint" type="fixed">
             <origin rpy="0 0 0" xyz="0.0 0.0 ${1.7 * robot_scale}"/>
             <parent link="airplane_link"/>
             <child link="lidar_link"/>
+        </joint>
+        <!-- IMU lidar joint-->
+        <joint name="imu_link_joint" type="fixed">
+            <origin rpy="0 0 0" xyz="0.0 0.0 0.0"/>
+            <parent link="airplane_link"/>
+            <child link="imu_link"/>
         </joint>
         <!-- Add a camera to follow the Airplane -->

File: ros_ws/src/uav_description/urdf/fixed_wing/airplane_gazebo.xacro (robot description, xacro)
@@ -4,5 +4,5 @@
     <xacro:property name="camera_noise_stddev" default="0.05"/>
     <!-- Define the vertical angular limit that the GNSS analize the multipath-->
-    <xacro:property name="max_gnss_lidar_ver" default="1.57"/>
+    <xacro:property name="max_gnss_lidar_ver" default="1.05"/>
     <xacro:macro name="airplane_sim" params="robot_name camera_num robot_scale world_name initial_alt">
         <!-- Add the frontal camera sensor -->
@@ -61,12 +61,12 @@
                     <scan>
                         <horizontal>
-                            <samples>6</samples>
-                            <resolution>1</resolution>
+                            <samples>4</samples>
+                            <resolution>0.5</resolution>
                             <min_angle>-3.1416</min_angle>
                             <max_angle>3.1416</max_angle>
                         </horizontal>
                         <vertical>
-                            <samples>6</samples>
-                            <resolution>1</resolution>
+                            <samples>2</samples>
+                            <resolution>0.5</resolution>
                             <min_angle>0</min_angle>
                             <max_angle>${max_gnss_lidar_ver}</max_angle>
@@ -75,6 +75,6 @@
                     <range>
                         <min>${(robot_scale * 10.0)}</min>
-                        <max>30.0</max>
-                        <resolution>0.2</resolution>
+                        <max>8.0</max>
+                        <resolution>1.5</resolution>
                     </range>
                 </ray>
@@ -97,4 +97,27 @@
             </plugin>
         </gazebo>
+        <!--IMU link that works as the ADS-B reciever-->
+        <gazebo reference="imu_link">
+            <sensor name="imu_sensor" type="imu">
+                <always_on>1</always_on>
+                <update_rate>100</update_rate>
+                <visualize>true</visualize>
+                <topic>${robot_name}/imu/out</topic>
+                <imu></imu>
+            </sensor>
+        </gazebo>
+        <gazebo>
+            <plugin filename="gz-sim-imu-system" name="gz::sim::systems::Imu">
+            </plugin>
+        </gazebo>
+        <gazebo>
+             <plugin name="adsb_plugin" filename="libadsb_plugin.so">
+                <topic>${robot_name}/imu/out</topic>
+                <cmdGNSSTopic>${robot_name}/gnss_multipath_fix</cmdGNSSTopic>
+                <frame_id>${robot_name}/base_link/imu_link</frame_id>
+                <cmdADSBTopic>${robot_name}/adsb_info</cmdADSBTopic>
+                <adsb_start_srv_stopic>${robot_name}/restart_adsb</adsb_start_srv_stopic>
+            </plugin>
+        </gazebo>
     </xacro:macro>
 </robot>
