Commit message: Refactor: Stop tracking flight data and add Dubins path logic

File: ros_ws/src/uav_description/urdf/vtol/vtol.xacro (robot description, xacro)
@@ -231,5 +231,5 @@
         <!-- Fixed joint to dummy link -->
         <joint name="vtol_joint" type="fixed">
-            <origin xyz="0.0 0.0 0.0" rpy="0.0 0.0 1.5708"/>
+            <origin xyz="0.0 0.0 0.0" rpy="0.0 0.0 0.0"/>
             <parent link="base_link"/>
             <child link="vtol_body"/>
